File: PS-LVDistributionPCB.kicad_pcb (KiCad board)
At the start: 2 copper layers, 6 parts, among them J1 Critical Power, J2 Non-Critical Power, J3 Power Conn, J4 Power Conn

Commit message: finished schematic
Parts:
- added D1: 20mA, LED_SMD:LED_0805_2012Metric, F.Cu at (26.9, 91.6)
- added D10: 20mA, LED_SMD:LED_0805_2012Metric, F.Cu at (30.5, 127.7)
- added D11: 20mA, LED_SMD:LED_0805_2012Metric, F.Cu at (30.5, 130.7)
- added D12: 20mA, LED_SMD:LED_0805_2012Metric, F.Cu at (30.5, 133.8)
- added D13: 20mA, LED_SMD:LED_0805_2012Metric, F.Cu at (30.5, 136.8)
- added D14: 20mA, LED_SMD:LED_0805_2012Metric, F.Cu at (30.9, 145.1)
- added D15: 20mA, LED_SMD:LED_0805_2012Metric, F.Cu at (34.1, 114.7)
- added D16: 20mA, LED_SMD:LED_0805_2012Metric, F.Cu at (34.1, 117.8)
- added D17: 20mA, LED_SMD:LED_0805_2012Metric, F.Cu at (35.0, 127.7)
- added D18: 20mA, LED_SMD:LED_0805_2012Metric, F.Cu at (35.0, 130.7)
- added D19: 20mA, LED_SMD:LED_0805_2012Metric, F.Cu at (35.0, 133.8)
- added D2: 20mA, LED_SMD:LED_0805_2012Metric, F.Cu at (26.9, 94.7)
- added D20: 20mA, LED_SMD:LED_0805_2012Metric, F.Cu at (74.2, 35.9)
- added D21: 20mA, LED_SMD:LED_0805_2012Metric, F.Cu at (48.8, 31.7)
- added D3: 20mA, LED_SMD:LED_0805_2012Metric, F.Cu at (26.9, 97.7)
- added D4: 20mA, LED_SMD:LED_0805_2012Metric, F.Cu at (26.9, 100.7)
- added D5: 20mA, LED_SMD:LED_0805_2012Metric, F.Cu at (26.9, 103.8)
- added D6: 20mA, LED_SMD:LED_0805_2012Metric, F.Cu at (26.9, 106.8)
- added D7: 20mA, LED_SMD:LED_0805_2012Metric, F.Cu at (26.9, 109.9)
- added D8: 20mA, LED_SMD:LED_0805_2012Metric, F.Cu at (29.6, 114.7)
- added D9: 20mA, LED_SMD:LED_0805_2012Metric, F.Cu at (29.6, 117.8)
- added F1: Fuse, footprints:3588, F.Cu at (141.6, 22.0)
- added F10: Fuse, footprints:3588, F.Cu at (105.0, 122.3)
- added F11: Fuse, footprints:3588, F.Cu at (32.5, 79.0)
- added F12: Fuse, footprints:3588, F.Cu at (32.5, 91.0)
- added F13: Fuse, footprints:3588, F.Cu at (32.5, 107.2)
- added F14: Fuse, footprints:3588, F.Cu at (28.2, 42.1)
- added F15: Fuse, footprints:3588, F.Cu at (100.8, 178.7)
- added F16: Fuse, footprints:3588, F.Cu at (100.8, 190.7)
- added F17: Fuse, footprints:3588, F.Cu at (72.3, 87.2)
- added F18: Fuse, footprints:3588, F.Cu at (98.0, 142.7)
- added F19: Fuse, footprints:3588, F.Cu at (133.1, 177.6)
- added F2: Fuse, footprints:3588, F.Cu at (187.5, 23.0)
- added F20: Fuse, footprints:3588, F.Cu at (133.1, 189.5)
- added F21: Fuse, footprints:3588, F.Cu at (97.0, 107.4)
- added F22: Fuse, footprints:3588, F.Cu at (69.8, 28.3)
- added F23: Fuse, footprints:3588, F.Cu at (37.0, 28.3)
- added F24: Fuse, footprints:3588, F.Cu at (37.0, 40.3)
- added F4: Fuse, footprints:3588, F.Cu at (141.6, 33.9)
- added F5: Fuse, footprints:3588, F.Cu at (141.6, 45.9)
- added F6: Fuse, footprints:3588, F.Cu at (141.6, 57.9)
- added F7: Fuse, footprints:3588, F.Cu at (141.6, 69.9)
- added F8: Fuse, footprints:3588, F.Cu at (141.6, 81.9)
- added F9: Fuse, footprints:3588, F.Cu at (141.6, 95.0)
- added J1: Non-Critical Power, footprints:Molex_Micro-Fit_3.0_43650-0215_1x02_P3.00mm_Vertical, F.Cu at (103.2, 126.9)
- added J10: Critical Power, footprints:Molex_Micro-Fit_3.0_43650-0215_1x02_P3.00mm_Vertical, F.Cu at (31.5, 187.9)
- added J11: Critical Power, footprints:Molex_Micro-Fit_3.0_43650-0215_1x02_P3.00mm_Vertical, F.Cu at (30.5, 46.7)
- added J12: Non-Critical Power, footprints:Molex_Micro-Fit_3.0_43650-0215_1x02_P3.00mm_Vertical, F.Cu at (103.1, 186.7)
- added J13: Non-Critical Power, footprints:Molex_Micro-Fit_3.0_43650-0215_1x02_P3.00mm_Vertical, F.Cu at (74.6, 86.6)
- added J14: Non-Critical Power, footprints:Molex_Micro-Fit_3.0_43650-0215_1x02_P3.00mm_Vertical, F.Cu at (73.5, 127.0)
- added J15: Non-Critical Power, footprints:Molex_Micro-Fit_3.0_43650-0215_1x02_P3.00mm_Vertical, F.Cu at (73.2, 148.2)
- added J16: Non-Critical Power, footprints:Molex_Micro-Fit_3.0_43650-0215_1x02_P3.00mm_Vertical, F.Cu at (74.5, 167.9)
- added J17: Non-Critical Power, footprints:Molex_Micro-Fit_3.0_43650-0215_1x02_P3.00mm_Vertical, F.Cu at (75.0, 188.1)
- added J18: Non-Critical Power, footprints:Molex_Micro-Fit_3.0_43650-0215_1x02_P3.00mm_Vertical, F.Cu at (104.3, 147.2)
- added J19: Non-Critical Power, footprints:Molex_Micro-Fit_3.0_43650-0215_1x02_P3.00mm_Vertical, F.Cu at (102.7, 167.2)
- added J20: Non-Critical Power, footprints:Molex_Micro-Fit_3.0_43650-0215_1x02_P3.00mm_Vertical, F.Cu at (103.3, 106.8)
- added J21: Non-Critical Power, Connector_Molex:Molex_Sabre_43160-0102_1x02_P7.49mm_Vertical, F.Cu at (73.0, 106.0)
- added J22: Critical Power, footprints:Molex_Micro-Fit_3.0_43650-0215_1x02_P3.00mm_Vertical, F.Cu at (64.6, 37.8)
- added J23: Power Conn, Connector_Molex:Molex_Sabre_43160-0102_1x02_P7.49mm_Vertical, F.Cu at (35.2, 56.8)
- added J24: Critical Power, footprints:Molex_Micro-Fit_3.0_43650-0215_1x02_P3.00mm_Vertical, F.Cu at (50.9, 25.9)
- added J3: Critical Power, footprints:Molex_Micro-Fit_3.0_43650-0215_1x02_P3.00mm_Vertical, F.Cu at (30.7, 87.0)
- added J4: Power Conn, Connector_Molex:Molex_Sabre_43160-0102_1x02_P7.49mm_Vertical, F.Cu at (182.3, 32.5)
- added J6: Critical Power, footprints:Molex_Micro-Fit_3.0_43650-0215_1x02_P3.00mm_Vertical, F.Cu at (30.7, 106.7)
- added J7: Critical Power, footprints:Molex_Micro-Fit_3.0_43650-0215_1x02_P3.00mm_Vertical, F.Cu at (31.7, 129.0)
- added J8: Critical Power, footprints:Molex_Micro-Fit_3.0_43650-0215_1x02_P3.00mm_Vertical, F.Cu at (32.0, 149.7)
- added J9: Critical Power, footprints:Molex_Micro-Fit_3.0_43650-0215_1x02_P3.00mm_Vertical, F.Cu at (31.5, 168.7)
- added R1: 505, Resistor_SMD:R_0805_2012Metric, F.Cu at (136.0, 112.0)
- added R10: 505, Resistor_SMD:R_0805_2012Metric, F.Cu at (140.9, 124.0)
- added R11: 505, Resistor_SMD:R_0805_2012Metric, F.Cu at (141.0, 129.0)
- added R12: 505, Resistor_SMD:R_0805_2012Metric, F.Cu at (141.0, 134.0)
- added R13: 505, Resistor_SMD:R_0805_2012Metric, F.Cu at (141.2, 140.0)
- added R14: 505, Resistor_SMD:R_0805_2012Metric, F.Cu at (141.2, 145.5)
- added R15: 505, Resistor_SMD:R_0805_2012Metric, F.Cu at (145.0, 112.0)
- added R16: 505, Resistor_SMD:R_0805_2012Metric, F.Cu at (145.0, 118.0)
- added R17: 505, Resistor_SMD:R_0805_2012Metric, F.Cu at (145.5, 124.0)
- added R18: 505, Resistor_SMD:R_0805_2012Metric, F.Cu at (145.5, 129.0)
- added R19: 505, Resistor_SMD:R_0805_2012Metric, F.Cu at (145.9, 134.0)
- added R2: 505, Resistor_SMD:R_0805_2012Metric, F.Cu at (135.5, 118.0)
- added R20: 505, Resistor_SMD:R_0805_2012Metric, F.Cu at (74.1, 38.9)
- added R21: 505, Resistor_SMD:R_0805_2012Metric, F.Cu at (53.2, 31.7)
- added R3: 505, Resistor_SMD:R_0805_2012Metric, F.Cu at (135.5, 124.0)
- added R4: 505, Resistor_SMD:R_0805_2012Metric, F.Cu at (135.5, 129.0)
- added R5: 505, Resistor_SMD:R_0805_2012Metric, F.Cu at (135.5, 134.0)
- added R6: 505, Resistor_SMD:R_0805_2012Metric, F.Cu at (135.5, 140.0)
- added R7: 505, Resistor_SMD:R_0805_2012Metric, F.Cu at (135.5, 145.5)
- added R8: 505, Resistor_SMD:R_0805_2012Metric, F.Cu at (140.5, 112.0)
- added R9: 505, Resistor_SMD:R_0805_2012Metric, F.Cu at (140.5, 118.5)
- J2: footprint Connector_Molex:Molex_Sabre_43160-0102_1x02_P7.49mm_Vertical -> footprints:Molex_Micro-Fit_3.0_43650-0215_1x02_P3.00mm_Vertical
- J5: renamed from J4; footprint footprints:Molex_Micro-Fit_3.0_43650-0215_1x02_P3.00mm_Vertical -> Connector_Molex:Molex_Sabre_43160-0102_1x02_P7.49mm_Vertical
- moved J1 106.9 mm to (30.0, 67.7)
- moved F1 65.3 mm to (224.7, 101.1)
- moved J3 65.3 mm to (219.5, 110.6)
- moved F3 64.0 mm to (186.5, 47.5)
- moved J5 64.0 mm to (181.3, 57.0)
- moved J2 37.5 mm to (102.3, 85.8)
- renumbered F2 to F3

Commit message: finished pcb
Parts:
- removed D21, D7: 20mA, LED_SMD:LED_0805_2012Metric
- removed the F1 at (141.6, 22.0)
- removed the F1 at (224.7, 101.1)
- removed F23, F24, F9: Fuse, footprints:3588
- removed the J1 at (103.2, 126.9)
- removed the J1 at (30.0, 67.7)
- removed J11, J24: Critical Power, footprints:Molex_Micro-Fit_3.0_43650-0215_1x02_P3.00mm_Vertical
- removed J23: Power Conn, Connector_Molex:Molex_Sabre_43160-0102_1x02_P7.49mm_Vertical
- removed the J3 at (30.7, 87.0)
- removed the J3 at (219.5, 110.6)
- removed R21, R7: 505, Resistor_SMD:R_0805_2012Metric
- added F1: 10A, footprints:3588, F.Cu at (180.5, 94.4)
- added J1: NON CRIT OUT, footprints:Molex_Micro-Fit_3.0_43650-0215_1x02_P3.00mm_Vertical, F.Cu at (100.8, 130.4)
- added J3: CRIT OUT, footprints:Molex_Micro-Fit_3.0_43650-0215_1x02_P3.00mm_Vertical, F.Cu at (179.0, 77.8)
- F10, F11, F12, F13, F14, F15, F16, F17, F18, F19, F2, F20, F22, F4, F5, F6, F7, F8: value Fuse -> 10A
- F21, F3: value Fuse -> 30A
- J10, J22, J6, J7, J8, J9: value Critical Power -> CRIT OUT
- J12, J13, J14, J15, J16, J17, J18, J19, J2, J20: value Non-Critical Power -> NON CRIT OUT
- J21: value Non-Critical Power -> CRIT; moved to B.Cu
- J4: value Power Conn -> NON CRIT OUT; footprint Connector_Molex:Molex_Sabre_43160-0102_1x02_P7.49mm_Vertical -> footprints:Molex_Micro-Fit_3.0_43650-0215_1x02_P3.00mm_Vertical
- J5: value Power Conn -> NON CRIT; moved to B.Cu
- moved D18 193.3 mm to (222.5, 84.0), turned to 180 degrees
- moved D17 183.5 mm to (218.5, 124.5)
- moved D19 181.0 mm to (209.0, 84.0), turned to 180 degrees
- moved D16 170.7 mm to (204.7, 124.5)
- moved D15 157.2 mm to (191.0, 124.5)
- moved F14 156.3 mm to (167.2, 113.6), turned to -90 degrees
- moved D1 155.4 mm to (182.1, 83.9), turned to 180 degrees
- moved D14 149.1 mm to (178.6, 124.5)
- moved J19 146.8 mm to (219.0, 77.5)
- moved J17 145.4 mm to (208.5, 130.4), turned to 180 degrees
- moved D2 142.5 mm to (169.0, 83.9), turned to 180 degrees
- moved J6 137.8 mm to (165.5, 77.9)
- moved F17 137.3 mm to (207.0, 113.5), turned to -90 degrees
- moved J10 135.9 mm to (111.5, 78.0)
- moved D13 135.1 mm to (165.1, 124.5)
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Connections:
- D1 pad 1: GND_A -> GND
- D10 pad 1: GND_B -> GND
- D11 pad 1: GND_B -> GND
- D12 pad 1: GND_B -> GND
- D13 pad 1: GND_B -> GND
- D14 pad 1: GND_B -> GND
- D15 pad 1: GND_B -> GND
- D16 pad 1: GND_B -> GND
- D17 pad 1: GND_B -> GND
- D18 pad 1: GND_B -> GND
- D19 pad 1: GND_B -> GND
- D2 pad 1: GND_A -> GND
- D20 pad 1: GND_A -> GND
- D3 pad 1: GND_A -> GND
- D4 pad 1: GND_A -> GND
- D5 pad 1: GND_A -> GND
- D6 pad 1: GND_A -> GND
- D8 pad 1: GND_B -> GND
- D9 pad 1: GND_B -> GND
- F10 pad 1: Net-(F10-Pad1) -> +12V_NON
- F10 pad 2: +12V_B -> Net-(J2-Pin_1)
- F11 pad 1: Net-(F10-Pad1) -> +12V_NON
- F11 pad 2: +12V_B -> Net-(J4-Pin_1)
- F12 pad 1: Net-(F10-Pad1) -> +12V_NON
- F12 pad 2: +12V_B -> Net-(J12-Pin_1)
- F13 pad 1: Net-(F10-Pad1) -> +12V_NON
- F13 pad 2: +12V_B -> Net-(J13-Pin_1)
- F14 pad 1: Net-(F10-Pad1) -> +12V_NON
- F14 pad 2: +12V_B -> Net-(J14-Pin_1)
- F15 pad 1: Net-(F10-Pad1) -> +12V_NON
- F15 pad 2: +12V_B -> Net-(J15-Pin_1)
- F16 pad 1: Net-(F10-Pad1) -> +12V_NON
- F16 pad 2: +12V_B -> Net-(J16-Pin_1)
- F17 pad 1: Net-(F10-Pad1) -> +12V_NON
- F17 pad 2: +12V_B -> Net-(J17-Pin_1)
- F18 pad 1: Net-(F10-Pad1) -> +12V_NON
- F18 pad 2: +12V_B -> Net-(J18-Pin_1)
- F19 pad 1: Net-(F10-Pad1) -> +12V_NON
- F19 pad 2: +12V_B -> Net-(J19-Pin_1)
- F2 pad 1: +12V_A -> +12V_NON
- F2 pad 2: Net-(J4-Pin_1) -> Net-(J1-Pin_1)
- F20 pad 1: Net-(F10-Pad1) -> +12V_NON
- F20 pad 2: +12V_B -> Net-(J20-Pin_1)
- F21 pad 1: Net-(F10-Pad1) -> +12V_CRIT
- F21 pad 2: +12V_B -> Net-(J21-Pin_1)
- F22 pad 1: unconnected-(F22-Pad1) -> +12V_CRIT
- F22 pad 2: +12V_A -> Net-(J22-Pin_1)
- F3 pad 1: +12V_B -> +12V_NON
- F4 pad 1: Net-(F1-Pad1) -> +12V_CRIT
- F4 pad 2: +12V_A -> Net-(J6-Pin_1)
- F5 pad 1: Net-(F1-Pad1) -> +12V_CRIT
- F5 pad 2: +12V_A -> Net-(J7-Pin_1)
- F6 pad 1: Net-(F1-Pad1) -> +12V_CRIT
- F6 pad 2: +12V_A -> Net-(J8-Pin_1)
- F7 pad 1: Net-(F1-Pad1) -> +12V_CRIT
- F7 pad 2: +12V_A -> Net-(J9-Pin_1)
- F8 pad 1: Net-(F1-Pad1) -> +12V_CRIT
- F8 pad 2: +12V_A -> Net-(J10-Pin_1)
- J10 pad 1: +12V_A -> Net-(J10-Pin_1)
- J10 pad 2: GND_A -> GND
- J12 pad 1: +12V_B -> Net-(J12-Pin_1)
- J12 pad 2: GND_B -> GND
- J13 pad 1: +12V_B -> Net-(J13-Pin_1)
- J13 pad 2: GND_B -> GND
- J14 pad 1: +12V_B -> Net-(J14-Pin_1)
- J14 pad 2: GND_B -> GND
- J15 pad 1: +12V_B -> Net-(J15-Pin_1)
- J15 pad 2: GND_B -> GND
- J16 pad 1: +12V_B -> Net-(J16-Pin_1)
- J16 pad 2: GND_B -> GND
- J17 pad 1: +12V_B -> Net-(J17-Pin_1)
- J17 pad 2: GND_B -> GND
- J18 pad 1: +12V_B -> Net-(J18-Pin_1)
- J18 pad 2: GND_B -> GND
- J19 pad 1: +12V_B -> Net-(J19-Pin_1)
- J19 pad 2: GND_B -> GND
- J2 pad 1: +12V_B -> Net-(J2-Pin_1)
- J2 pad 2: GND_B -> GND
- J20 pad 1: +12V_B -> Net-(J20-Pin_1)
- J20 pad 2: GND_B -> GND
- J21 pad 1: +12V_B -> Net-(J21-Pin_1)
- J21 pad 2: GND_B -> GND
- J22 pad 1: +12V_A -> Net-(J22-Pin_1)
- J22 pad 2: GND_A -> GND
- J4 pad 2: GND_A -> GND
- J5 pad 2: GND_B -> GND
- J6 pad 1: +12V_A -> Net-(J6-Pin_1)
- J6 pad 2: GND_A -> GND
- J7 pad 1: +12V_A -> Net-(J7-Pin_1)
- J7 pad 2: GND_A -> GND
- J8 pad 1: +12V_A -> Net-(J8-Pin_1)
- J8 pad 2: GND_A -> GND
- J9 pad 1: +12V_A -> Net-(J9-Pin_1)
- J9 pad 2: GND_A -> GND
- R1 pad 1: +12V_A -> Net-(J3-Pin_1)
- R10 pad 1: +12V_B -> Net-(J4-Pin_1)
- R11 pad 1: +12V_B -> Net-(J12-Pin_1)
- R12 pad 1: +12V_B -> Net-(J13-Pin_1)
- R13 pad 1: +12V_B -> Net-(J14-Pin_1)
- R14 pad 1: +12V_B -> Net-(J15-Pin_1)
- R15 pad 1: +12V_B -> Net-(J16-Pin_1)
- R16 pad 1: +12V_B -> Net-(J17-Pin_1)
- R17 pad 1: +12V_B -> Net-(J18-Pin_1)
- R18 pad 1: +12V_B -> Net-(J19-Pin_1)
- R19 pad 1: +12V_B -> Net-(J20-Pin_1)
- R2 pad 1: +12V_A -> Net-(J6-Pin_1)
- R20 pad 1: +12V_A -> Net-(J22-Pin_1)
- R3 pad 1: +12V_A -> Net-(J7-Pin_1)
- R4 pad 1: +12V_A -> Net-(J8-Pin_1)
- R5 pad 1: +12V_A -> Net-(J9-Pin_1)
- R6 pad 1: +12V_A -> Net-(J10-Pin_1)
- R8 pad 1: +12V_B -> Net-(J1-Pin_1)
- R9 pad 1: +12V_B -> Net-(J2-Pin_1)
Routing:
- net GND: track 0.00 -> 124.8 mm
- net Net-(J21-Pin_1): track 0.00 -> 23.9 mm
- net Net-(J5-Pin_1): track 0.00 -> 23.5 mm
- net Net-(J20-Pin_1): track 0.00 -> 19.1 mm
- net Net-(J19-Pin_1): track 0.00 -> 19.1 mm
- net Net-(J18-Pin_1): track 0.00 -> 19.0 mm
- net Net-(J4-Pin_1): track 0.00 -> 18.9 mm
- net Net-(J3-Pin_1): track 0.00 -> 18.9 mm
- net Net-(J12-Pin_1): track 0.00 -> 18.9 mm
- net Net-(J15-Pin_1): track 0.00 -> 18.8 mm
- net Net-(J13-Pin_1): track 0.00 -> 18.8 mm
- net Net-(J1-Pin_1): track 0.00 -> 18.7 mm
- net Net-(J6-Pin_1): track 0.00 -> 18.7 mm
- net Net-(J14-Pin_1): track 0.00 -> 18.7 mm
- net Net-(J2-Pin_1): track 0.00 -> 18.7 mm
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- added copper zone on F.Cu, net +12V_CRIT
- added copper zone on F.Cu, net +12V_NON
- added copper zone on B.Cu, net GND
Other:
- board outline added: 161 x 63 mm

Commit message: more fill zones
Parts:
- moved D1 4.61 mm to (186.6, 82.9)
- moved D10 4.61 mm to (129.1, 123.5)
- moved D11 4.61 mm to (142.6, 123.5)
- moved D12 4.61 mm to (156.1, 123.5)
- moved D13 4.61 mm to (169.6, 123.5)
- moved D14 4.61 mm to (183.1, 123.5)
- moved D15 4.61 mm to (195.5, 123.5)
- moved D16 4.61 mm to (209.2, 123.5)
- moved D17 4.61 mm to (223.0, 123.5)
- moved D18 4.61 mm to (227.0, 83.0)
- moved D19 4.61 mm to (213.5, 83.0)
- moved D2 4.61 mm to (173.5, 82.9)
- moved D20 4.61 mm to (106.0, 82.9)
- moved D3 4.61 mm to (160.1, 82.9)
- moved D4 4.61 mm to (146.4, 82.9)
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Routing:
- net Net-(J4-Pin_1): track 18.9 -> 0.00 mm
- net Net-(J3-Pin_1): track 18.9 -> 0.00 mm
- net Net-(J12-Pin_1): track 18.9 -> 0.00 mm
- net Net-(J13-Pin_1): track 18.8 -> 0.00 mm
- net Net-(J6-Pin_1): track 18.7 -> 0.00 mm
- net Net-(J8-Pin_1): track 18.6 -> 0.00 mm
- net Net-(J15-Pin_1): track 18.8 -> 0.15 mm
- net Net-(J20-Pin_1): track 19.1 -> 0.46 mm
- net Net-(J19-Pin_1): track 19.1 -> 0.46 mm
- net Net-(J1-Pin_1): track 18.7 -> 0.18 mm
- net Net-(J17-Pin_1): track 18.6 -> 0.04 mm
- net Net-(J2-Pin_1): track 18.7 -> 0.10 mm
- net Net-(J14-Pin_1): track 18.7 -> 0.15 mm
- net Net-(J18-Pin_1): track 19.0 -> 0.54 mm
- net Net-(J22-Pin_1): track 18.4 -> 0.00 mm
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- added copper zone on F.Cu, net Net-(J1-Pin_1)
- added copper zone on F.Cu, net Net-(J10-Pin_1)
- added copper zone on F.Cu, net Net-(J12-Pin_1)
- added copper zone on F.Cu, net Net-(J13-Pin_1)
- added copper zone on F.Cu, net Net-(J14-Pin_1)
- added copper zone on F.Cu, net Net-(J15-Pin_1)
- added copper zone on F.Cu, net Net-(J16-Pin_1)
- added copper zone on F.Cu, net Net-(J17-Pin_1)
- added copper zone on F.Cu, net Net-(J18-Pin_1)
- added copper zone on F.Cu, net Net-(J19-Pin_1)
- added copper zone on F.Cu, net Net-(J2-Pin_1)
- added copper zone on F.Cu, net Net-(J20-Pin_1)
- added copper zone on F.Cu, net Net-(J22-Pin_1)
- added copper zone on F.Cu, net Net-(J3-Pin_1)
- added copper zone on F.Cu, net Net-(J4-Pin_1)
- added copper zone on F.Cu, net Net-(J6-Pin_1)
- added copper zone on F.Cu, net Net-(J7-Pin_1)
- added copper zone on F.Cu, net Net-(J8-Pin_1)
- added copper zone on F.Cu, net Net-(J9-Pin_1)
Other:
- outline, holes or cut-outs redrawn
