File: noncriticalpwr.kicad_sch (KiCad schematic)
At the start: 6 parts

Commit message: solder bridges
Parts:
- added JP20: SolderJumper_2_Open, Jumper:SolderJumper-2_P1.3mm_Open_TrianglePad1.0x1.5mm, symbol Jumper:SolderJumper_2_Open
- renumbered NC_D9 to NC_D1, NC_F9 to NC_F1, NC_J9 to NC_J1, NC_R17 to NC_R1, NC_R18 to NC_R2, NC_U9 to NC_U1
Connections:
- net at NC_R1.2: now also JP20.1 (A); no longer NC_U1.1
- new net: JP20.2 (B), NC_U1.1
Changed lines of the file:
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@@
 (kicad_sch
-	(version 20231120)
+	(version 20250114)
 	(generator "eeschema")
-	(generator_version "8.0")
+	(generator_version "9.0")
 	(paper "A4")
 	(junction
@@
 	(wire
 		(pts
-			(xy 50.8 34.29) (xy 50.8 44.45)
+			(xy 50.8 34.29) (xy 50.8 35.56)
 		)
 		(stroke
@@
 		(pts
 			(xy 83.82 54.61) (xy 83.82 58.42)
+		)
+		(stroke
+			(width 0)
+			(type default)
+		)
+	)
+	(wire
+		(pts
+			(xy 50.8 43.18) (xy 50.8 44.45)
 		)
 		(stroke
@@
 		(dnp no)
 		(fields_autoplaced yes)
-		(property "Reference" "NC_R18"
+		(property "Reference" "NC_R2"
 			(at 86.36 33.0199 0)
 			(effects
@@
 		(on_board yes)
 		(dnp no)
-		(property "Reference" "#PWR036"
+		(property "Reference" "#PWR02"
 			(at 67.31 66.04 0)
 			(effects
@@
 		(on_board yes)
 		(dnp no)
-		(property "Reference" "NC_J9"
+		(property "Reference" "NC_J1"
 			(at 101.6 16.51 90)
 			(effects
@@
 		(on_board yes)
 		(dnp no)
-		(property "Reference" "NC_D9"
+		(property "Reference" "NC_D1"
 			(at 87.884 46.99 0)
 			(effects
@@
 				(path "/bae4e46c-28ae-4193-a5e0-928c081802f5/e148df88-9647-4e60-9f2c-a8647da26d9f"
 					(reference "NC_D11")
+					(unit 1)
+				)
+			)
+		)
+	)
+	(symbol
+		(lib_id "Jumper:SolderJumper_2_Open")
+		(at 50.8 39.37 270)
+		(unit 1)
+		(exclude_from_sim no)
+		(in_bom no)
+		(on_board yes)
+		(dnp no)
+		(property "Reference" "JP20"
+			(at 48.006 38.354 90)
+			(effects
+				(font
+					(size 1.27 1.27)
+				)
+				(justify right)
+			)
+		)
+		(property "Value" "SolderJumper_2_Open"
+			(at 48.006 40.64 90)
+			(effects
+				(font
+					(size 1.27 1.27)
+				)
+				(justify right)
+			)
+		)
+		(property "Footprint" "Jumper:SolderJumper-2_P1.3mm_Open_TrianglePad1.0x1.5mm"
+			(at 50.8 39.37 0)
+			(effects
+				(font
+					(size 1.27 1.27)
+				)
+				(hide yes)
+			)
+		)
+		(property "Datasheet" "~"
+			(at 50.8 39.37 0)
+			(effects
+				(font
+					(size 1.27 1.27)
+				)
+				(hide yes)
+			)
+		)
+		(property "Description" "Solder Jumper, 2-pole, open"
+			(at 50.8 39.37 0)
+			(effects
+				(font
+					(size 1.27 1.27)
+				)
+				(hide yes)
+			)
+		)
+		(pin "2"
+		)
+		(pin "1"
+		)
+		(instances
+			(project ""
+				(path "/bae4e46c-28ae-4193-a5e0-928c081802f5/24c2380e-3122-4ed4-8f93-9bbbae8c25de"
+					(reference "JP28")
+					(unit 1)
+				)
+				(path "/bae4e46c-28ae-4193-a5e0-928c081802f5/263de9e2-9bcb-44c7-bb7d-d3bf366c066d"
+					(reference "JP23")
+					(unit 1)
+				)
+				(path "/bae4e46c-28ae-4193-a5e0-928c081802f5/4704c24a-927d-4e3d-9a25-eccf94f40fd3"
+					(reference "JP26")
+					(unit 1)
+				)
+				(path "/bae4e46c-28ae-4193-a5e0-928c081802f5/4763536e-7ebc-46be-a770-f6b090c90a7e"
+					(reference "JP29")
+					(unit 1)
+				)
+				(path "/bae4e46c-28ae-4193-a5e0-928c081802f5/51321fa4-7e7d-4384-9966-2731239abadf"
+					(reference "JP21")
+					(unit 1)
+				)
+				(path "/bae4e46c-28ae-4193-a5e0-928c081802f5/52d1015b-6151-4c78-82f1-6085843c475d"
+					(reference "JP31")
+					(unit 1)
+				)
+				(path "/bae4e46c-28ae-4193-a5e0-928c081802f5/614c3992-1675-48b5-b9e3-8a437289e9ef"
+					(reference "JP27")
+					(unit 1)
+				)
+				(path "/bae4e46c-28ae-4193-a5e0-928c081802f5/85f611f4-5816-48a5-a428-9e0e856db9ae"
+					(reference "JP22")
+					(unit 1)
+				)
+				(path "/bae4e46c-28ae-4193-a5e0-928c081802f5/a857b892-d7fd-4dcd-80cf-5632ad5dd0c2"
+					(reference "JP25")
+					(unit 1)
+				)
+				(path "/bae4e46c-28ae-4193-a5e0-928c081802f5/be52c217-f59c-49b0-8ebd-705c7dac3fae"
+					(reference "JP24")
+					(unit 1)
+				)
+				(path "/bae4e46c-28ae-4193-a5e0-928c081802f5/c4f4a294-58a7-4e12-a3d4-c82fa063be77"
+					(reference "JP20")
+					(unit 1)
+				)
+				(path "/bae4e46c-28ae-4193-a5e0-928c081802f5/e148df88-9647-4e60-9f2c-a8647da26d9f"
+					(reference "JP30")
 					(unit 1)
 				)
@@
 		(on_board yes)
 		(dnp no)
-		(property "Reference" "NC_U9"
+		(property "Reference" "NC_U1"
 			(at 60.96 55.0418 0)
 			(effects
@@
 		(on_board yes)
 		(dnp no)
-		(property "Reference" "NC_F9"
+		(property "Reference" "NC_F1"
 			(at 41.91 20.574 90)
 			(effects
@@
 		(on_board yes)
 		(dnp no)
-		(property "Reference" "#PWR051"
+		(property "Reference" "#PWR043"
 			(at 96.52 38.1 0)
 			(effects
@@
 		(dnp no)
 		(fields_autoplaced yes)
-		(property "Reference" "NC_R17"
+		(property "Reference" "NC_R1"
 			(at 53.34 29.2099 0)
 			(effects
