File: MX150_Test_Board/MX150_Test_Board/MX150_Test_Board.kicad_pcb (KiCad board)
At the start: 2 copper layers, 81.5 x 59.7 mm, 8 parts, among them J1 MX150_02x03_Vertical, J2 MX150_02x04_Vertical, J3 MX150_02x08_Vertical, J4 MX150_02x10_Vertical, J5 MX150_02x04_RightAngle, J6 MX150_02x08_RightAngle, J7 MX150_02x10_RightAngle

Commit message: updated symbols
Parts:
- moved LOGO1 11.9 mm to (166.7, 100.7)
- moved J5 3.73 mm to (148.5, 98.4)
- moved J3 1.93 mm to (114.7, 100.8)
Other:
- board text added: "MX150 Test Board Surabhi K LHRS 2025"
Changed lines of the file:
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@@
 	(net 5 "unconnected-(J5-+24V-Pad1)")
 	(net 6 "unconnected-(J5-CANL_OUT-Pad7)")
-	(net 7 "unconnected-(J5-PWR_OUT*-Pad4)")
+	(net 7 "unconnected-(J2-24V_OUT*-Pad4)")
 	(net 8 "unconnected-(J5-CANH_IN-Pad2)")
 	(net 9 "unconnected-(J1-CANH_IN-Pad2)")
@@
 	(net 15 "unconnected-(J2-CANH_IN-Pad2)")
 	(net 16 "unconnected-(J2-+24V-Pad1)")
-	(net 17 "unconnected-(J2-PWR_OUT*-Pad4)")
+	(net 17 "unconnected-(J3-24V_OUT*-Pad4)")
 	(net 18 "unconnected-(J2-CANH_OUT-Pad6)")
 	(net 19 "unconnected-(J2-CANL_IN-Pad3)")
@@
 	(net 36 "unconnected-(J3-CANL_IN-Pad3)")
 	(net 37 "unconnected-(J3-Pad15)")
-	(net 38 "unconnected-(J3-PWR_OUT*-Pad4)")
+	(net 38 "unconnected-(J4-24V_OUT*-Pad4)")
 	(net 39 "unconnected-(J4-Pad10)")
 	(net 40 "unconnected-(J4-GND_OUT*-Pad14)")
@@
 	(net 55 "unconnected-(J4-CANL_IN-Pad3)")
 	(net 56 "unconnected-(J4-CANH_IN-Pad2)")
-	(net 57 "unconnected-(J4-PWR_OUT*-Pad4)")
+	(net 57 "unconnected-(J5-24V_OUT*-Pad4)")
 	(net 58 "unconnected-(J4-CANH_OUT-Pad12)")
 	(net 59 "unconnected-(J6-CANL_OUT-Pad11)")
@@
 	(net 66 "unconnected-(J6-Pad6)")
 	(net 67 "unconnected-(J6-Pad15)")
-	(net 68 "unconnected-(J6-PWR_OUT*-Pad4)")
+	(net 68 "unconnected-(J6-24V_OUT*-Pad4)")
 	(net 69 "unconnected-(J6-Pad14)")
 	(net 70 "unconnected-(J6-Pad16)")
@@
 	(net 75 "unconnected-(J7-Pad18)")
 	(net 76 "unconnected-(J7-Pad20)")
-	(net 77 "unconnected-(J7-PWR_OUT*-Pad4)")
+	(net 77 "unconnected-(J7-24V_OUT*-Pad4)")
 	(net 78 "unconnected-(J7-Pad6)")
 	(net 79 "unconnected-(J7-Pad16)")
@@
 	(footprint "UTSVT_Logos:LHRs_LOGO"
 		(layer "F.Cu")
-		(at 157 107.6)
+		(at 166.7 100.7)
 		(property "Reference" "LOGO1"
 			(at 2.286 8.128 0)
@@
 	(footprint "UTSVT_Connectors:CONN_SD-75900-001_2X04_MOL"
 		(layer "F.Cu")
-		(at 152.228549 98.400003 180)
+		(at 148.500001 98.400003 180)
 		(tags "759001141 ")
 		(property "Reference" "J5"
@@
 			)
 		)
+		(property "P/N" "759001141"
+			(at 0 0 180)
+			(unlocked yes)
+			(layer "F.Fab")
+			(hide yes)
+			(effects
+				(font
+					(size 1 1)
+					(thickness 0.15)
+				)
+			)
+		)
 		(sheetname "/")
 		(sheetfile "MX150_Test_Board.kicad_sch")
@@
 			(layers "*.Cu" "*.Mask")
 			(remove_unused_layers no)
-			(net 7 "unconnected-(J5-PWR_OUT*-Pad4)")
-			(pinfunction "PWR_OUT*")
+			(net 57 "unconnected-(J5-24V_OUT*-Pad4)")
+			(pinfunction "24V_OUT*")
 			(pintype "bidirectional+no_connect")
 		)
@@
 			)
 		)
+		(property "P/N" "757575131"
+			(at 0 0 0)
+			(unlocked yes)
+			(layer "F.Fab")
+			(hide yes)
+			(effects
+				(font
+					(size 1 1)
+					(thickness 0.15)
+				)
+			)
+		)
 		(sheetname "/")
 		(sheetfile "MX150_Test_Board.kicad_sch")
@@
 			)
 		)
+		(property "P/N" "757575101"
+			(at 0 0 0)
+			(unlocked yes)
+			(layer "F.Fab")
+			(hide yes)
+			(effects
+				(font
+					(size 1 1)
+					(thickness 0.15)
+				)
+			)
+		)
 		(sheetname "/")
 		(sheetfile "MX150_Test_Board.kicad_sch")
@@
 			(layers "*.Cu" "*.Mask")
 			(remove_unused_layers no)
-			(net 57 "unconnected-(J4-PWR_OUT*-Pad4)")
-			(pinfunction "PWR_OUT*")
+			(net 38 "unconnected-(J4-24V_OUT*-Pad4)")
+			(pinfunction "24V_OUT*")
 			(pintype "bidirectional+no_connect")
 		)
@@
 			)
 		)
+		(property "P/N" "757575141"
+			(at 0 0 270)
+			(unlocked yes)
+			(layer "F.Fab")
+			(hide yes)
+			(effects
+				(font
+					(size 1 1)
+					(thickness 0.15)
+				)
+			)
+		)
 		(sheetname "/")
 		(sheetfile "MX150_Test_Board.kicad_sch")
@@
 			(layers "*.Cu" "*.Mask")
 			(remove_unused_layers no)
-			(net 17 "unconnected-(J2-PWR_OUT*-Pad4)")
-			(pinfunction "PWR_OUT*")
+			(net 7 "unconnected-(J2-24V_OUT*-Pad4)")
+			(pinfunction "24V_OUT*")
 			(pintype "bidirectional+no_connect")
 		)
@@
 	(footprint "UTSVT_Connectors:CONN16_0757575481_MOL"
 		(layer "F.Cu")
-		(at 116.5797 100.800599 180)
+		(at 114.65 100.800599 180)
 		(tags "757575481 ")
 		(property "Reference" "J3"
@@
 			)
 		)
+		(property "P/N" "757575481"
+			(at 0 0 180)
+			(unlocked yes)
+			(layer "F.Fab")
+			(hide yes)
+			(effects
+				(font
+					(size 1 1)
+					(thickness 0.15)
+				)
+			)
+		)
 		(sheetname "/")
 		(sheetfile "MX150_Test_Board.kicad_sch")
@@
 			(layers "*.Cu" "*.Mask")
 			(remove_unused_layers no)
-			(net 38 "unconnected-(J3-PWR_OUT*-Pad4)")
-			(pinfunction "PWR_OUT*")
+			(net 17 "unconnected-(J3-24V_OUT*-Pad4)")
+			(pinfunction "24V_OUT*")
 			(pintype "bidirectional+no_connect")
 		)
@@
 			)
 		)
+		(property "P/N" "759001101"
+			(at 0 0 0)
+			(unlocked yes)
+			(layer "F.Fab")
+			(hide yes)
+			(effects
+				(font
+					(size 1 1)
+					(thickness 0.15)
+				)
+			)
+		)
 		(sheetname "/")
 		(sheetfile "MX150_Test_Board.kicad_sch")
@@
 			(layers "*.Cu" "*.Mask")
 			(remove_unused_layers no)
-			(net 77 "unconnected-(J7-PWR_OUT*-Pad4)")
-			(pinfunction "PWR_OUT*")
+			(net 77 "unconnected-(J7-24V_OUT*-Pad4)")
+			(pinfunction "24V_OUT*")
 			(pintype "bidirectional+no_connect")
 		)
@@
 			)
 		)
+		(property "P/N" "759001181"
+			(at 0 0 90)
+			(unlocked yes)
+			(layer "F.Fab")
+			(hide yes)
+			(effects
+				(font
+					(size 1 1)
+					(thickness 0.15)
+				)
+			)
+		)
 		(sheetname "/")
 		(sheetfile "MX150_Test_Board.kicad_sch")
@@
 			(layers "*.Cu" "*.Mask")
 			(remove_unused_layers no)
-			(net 68 "unconnected-(J6-PWR_OUT*-Pad4)")
-			(pinfunction "PWR_OUT*")
+			(net 68 "unconnected-(J6-24V_OUT*-Pad4)")
+			(pinfunction "24V_OUT*")
 			(pintype "bidirectional+no_connect")
 		)
@@
 		(layer "Edge.Cuts")
 	)
+	(gr_text "MX150 Test Board\nSurabhi K LHRS 2025"
+		(at 159.5 98.5 0)
+		(layer "F.SilkS")
+		(effects
+			(font
+				(size 1 1)
+				(thickness 0.15)
+			)
+			(justify left bottom)
+		)
+	)
 	(embedded_fonts no)
