File: LV-Distribution/PS-LVDistributionPCB.kicad_pcb (KiCad board)
At the start: 2 copper layers, 132.1 x 58.5 mm, 42 parts, among them J1 Conn_01x02, J10 Conn_01x02, J11 Conn_01x02, J12 Conn_01x02, J15 Conn_01x20, J2 Conn_01x02, J3 Conn_01x02, J4 Conn_01x02, J5 Conn_01x02, J6 Conn_01x02, J7 Conn_01x02, J8 Conn_01x02, J9 Conn_01x02

Commit message: redo traces trial 1
Parts:
- removed J15: Conn_01x20, footprints:CONN_SD-34829-001_20_ST_MOL
- added D14: TVS, Diode_SMD:D_0603_1608Metric, F.Cu at (209.4, 95.4)
- added D7: TVS, Diode_SMD:D_0603_1608Metric, F.Cu at (209.4, 78.0)
- added F14: 3568, footprints:FUSE_3568, F.Cu at (216.2, 99.9)
- added F7: 3568, footprints:FUSE_3568, F.Cu at (216.2, 82.5)
- added J14: Conn_01x02, footprints:AMASS_XT30UPB-M_1x02_P5.0mm_Vertical, F.Cu at (213.7, 91.9)
- added J16: MX150_02x10_RightAngle, UTSVT_Connectors:CONN_SD-75900-001_2X10_MOL, B.Cu at (127.4, 167.3)
- added J17: MX150_02x10_RightAngle, footprints:CONN_SD-34829-001_20_ST_MOL, B.Cu at (95.1, 103.0)
- added J7: Conn_01x02, footprints:AMASS_XT30UPB-M_1x02_P5.0mm_Vertical, F.Cu at (213.7, 74.5)
- moved H2 18.5 mm to (233.1, 61.5)
- moved H4 18.5 mm to (233.1, 113.0)
- moved H5 18.5 mm to (233.1, 87.3)
- renumbered D9 to D10, D10 to D11, D11 to D12, D12 to D13, D7 to D8, D8 to D9, F9 to F10, F10 to F11, F11 to F12, F12 to F13, F7 to F8, F8 to F9, J9 to J10, J10 to J11, J11 to J12, J12 to J13, J7 to J8, J8 to J9
Connections:
- D10 pad 2: P9 -> P10
- D11 pad 2: P10 -> P11
- D12 pad 2: P11 -> P12
- D13 pad 2: P12 -> P13
- D8 pad 2: P7 -> P8
- D9 pad 2: P8 -> P9
- F10 pad 1: P9 -> P10
- F10 pad 3: P9 -> P10
- F11 pad 1: P10 -> P11
- F11 pad 3: P10 -> P11
- F12 pad 1: P11 -> P12
- F12 pad 2: Net-(J11-Pin_1) (its old number) -> Net-(J13-Pin_1)
- F12 pad 3: P11 -> P12
- F12 pad 4: Net-(J11-Pin_1) (its old number) -> Net-(J13-Pin_1)
- F13 pad 1: P12 -> P13
- F13 pad 3: P12 -> P13
- F8 pad 1: P7 -> P8
- F8 pad 3: P7 -> P8
- F9 pad 1: P8 -> P9
- F9 pad 3: P8 -> P9
- J12 pad 1: Net-(J11-Pin_1) (its old number) -> Net-(J12-Pin_1)
- J13 pad 1: Net-(J12-Pin_1) -> Net-(J13-Pin_1)
Routing:
- net P14: track 0.00 -> 147.7 mm
- net P13: track 0.00 -> 139.7 mm
- net P7: track 27.5 -> 119.6 mm
- net P10: track 89.0 -> 54.9 mm
- net P9: track 67.7 -> 37.8 mm
- net P8: track 47.5 -> 20.1 mm
- net (no net): track 0.00 -> 26.9 mm
- net P5: track 108.9 -> 89.8 mm
- net P2: track 60.8 -> 42.1 mm
- net P3: track 77.4 -> 58.8 mm
- net P6: track 125.8 -> 108.1 mm
- net P4: track 93.5 -> 75.8 mm
- net P11: track 93.3 -> 107.8 mm
- net Net-(J12-Pin_1): track 13.4 -> 0.00 mm
- net Net-(J11-Pin_1) (its old number): track 13.4 -> 0.00 mm
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Other:
- board size 132.1 x 58.5 mm -> 150.6 x 58.5 mm

Commit message: better layout but weird 3d stuff
Parts:
- removed J16: MX150_02x10_RightAngle, UTSVT_Connectors:CONN_SD-75900-001_2X10_MOL
- moved D1 1.10 mm to (104.4, 76.9), turned to 180 degrees
- moved D2 1.10 mm to (121.9, 76.9), turned to 180 degrees
- moved D3 1.10 mm to (139.4, 76.9), turned to 180 degrees
- moved D4 1.10 mm to (156.9, 76.9), turned to 180 degrees
- moved D5 1.10 mm to (174.4, 76.9), turned to 180 degrees
- moved D6 1.10 mm to (191.9, 76.9), turned to 180 degrees
- moved D7 1.10 mm to (209.4, 76.9), turned to 180 degrees
- moved F1 1.10 mm to (111.2, 81.4)
- moved F2 1.10 mm to (128.7, 81.4)
- moved F3 1.10 mm to (146.2, 81.4)
- moved F4 1.10 mm to (163.7, 81.4)
- moved F5 1.10 mm to (181.2, 81.4)
- moved F6 1.10 mm to (198.7, 81.4)
- moved F7 1.10 mm to (216.2, 81.4)
- moved J1 1.10 mm to (108.7, 73.4)
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Connections:
- F12 pad 2: Net-(J13-Pin_1) -> Net-(J12-Pin_1)
- F12 pad 4: Net-(J13-Pin_1) -> Net-(J12-Pin_1)
- F13 pad 2: Net-(J12-Pin_1) -> Net-(J13-Pin_1)
- F13 pad 4: Net-(J12-Pin_1) -> Net-(J13-Pin_1)
- J17 pad 1: P1 -> P3
- J17 pad 11: P11 -> P4
- J17 pad 12: P12 -> P5
- J17 pad 13: P13 -> GND
- J17 pad 14: P14 -> GND
- J17 pad 19: GND -> P12
- J17 pad 20: GND -> P11
- J17 pad 3: P3 -> P1
- J17 pad 4: P4 -> P6
- J17 pad 5: P5 -> P7
- J17 pad 6: P6 -> P14
- J17 pad 7: P7 -> P13
Routing:
- net GND: track 0.00 -> 198.0 mm
- net P13: track 139.7 -> 108.0 mm
- net P11: track 107.8 -> 77.9 mm
- net (no net): track 26.9 -> 0.00 mm
- net P14: track 147.7 -> 125.5 mm
- net P12: track 121.3 -> 102.8 mm
- net Net-(J7-Pin_1): track 0.00 -> 13.5 mm
- net Net-(J14-Pin_1): track 0.00 -> 13.5 mm
- net Net-(J13-Pin_1): track 0.00 -> 13.4 mm
- net Net-(J12-Pin_1): track 0.00 -> 13.4 mm
- net P5: track 89.8 -> 102.2 mm
- net P7: track 119.6 -> 125.5 mm
- net P1: track 24.0 -> 19.1 mm
- net P8: track 20.1 -> 15.8 mm
- net P2: track 42.1 -> 39.0 mm
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- added copper zone on B.Cu, net GND
- removed copper zone on F.Cu, net GND
Other:
- board size 150.6 x 58.5 mm -> 150.7 x 65 mm

Commit message: fixed 3d + gerbers
Parts:
- moved H2 1.70 mm to (231.4, 61.5)
- moved H4 1.70 mm to (231.4, 113.0)
- moved H5 1.70 mm to (231.4, 87.3)
Other:
- board size 150.7 x 65 mm -> 149 x 58.5 mm
Changed lines of the file:
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@@
 	(footprint "MountingHole:MountingHole_3.2mm_M3"
 		(layer "F.Cu")
-		(at 233.1 87.3)
+		(at 231.4 87.3)
 		(descr "Mounting Hole 3.2mm, no annular, M3")
 		(tags "mounting hole 3.2mm no annular m3")
@@
 	(footprint "MountingHole:MountingHole_3.2mm_M3"
 		(layer "F.Cu")
-		(at 233.1 61.5)
+		(at 231.4 61.5)
 		(descr "Mounting Hole 3.2mm, no annular, M3")
 		(tags "mounting hole 3.2mm no annular m3")
@@
 	(footprint "MountingHole:MountingHole_3.2mm_M3"
 		(layer "F.Cu")
-		(at 233.1 113)
+		(at 231.4 113)
 		(descr "Mounting Hole 3.2mm, no annular, M3")
 		(tags "mounting hole 3.2mm no annular m3")
@@
 		)
 		(fp_line
+			(start -16.660395 -9.152805)
+			(end 48.160405 -9.152805)
+			(stroke
+				(width 0.0254)
+				(type solid)
+			)
+			(layer "B.SilkS")
+		)
+		(fp_line
 			(start 48.287405 -8.845255)
 			(end 48.287405 0.677)
@@
 		)
 		(fp_line
-			(start -16.660395 -9.152805)
-			(end 48.160405 -9.152805)
-			(stroke
-				(width 0.0254)
-				(type solid)
-			)
-			(layer "Edge.Cuts")
-		)
-		(fp_line
 			(start 48.414405 -42.274404)
 			(end 48.414405 1.282701)
@@
 				(name "0348302001.stp")
 				(type model)
-				(checksum "9310518C80B9A11C3C709B68A6EC8CDD")
+				(checksum "03A4D46CEC60E7FBAAF483EA678A442B")
 			)
 		)
 		(model "kicad-embed://0348302001.stp"
 			(offset
-				(xyz -2.25 -8 -3)
+				(xyz -2.25 -8 -2.5)
 			)
 			(scale
@@
 		)
 	)
-	(gr_rect
-		(start 85.9 54.8)
-		(end 236.6 119.8)
+	(gr_line
+		(start 88.907196 58)
+		(end 231.907196 58)
+		(stroke
+			(width 0.2)
+			(type default)
+		)
+		(layer "Edge.Cuts")
+	)
+	(gr_line
+		(start 234.907196 61)
+		(end 234.907196 113.5)
+		(stroke
+			(width 0.2)
+			(type default)
+		)
+		(layer "Edge.Cuts")
+	)
+	(gr_line
+		(start 231.907196 116.5)
+		(end 88.907196 116.5)
+		(stroke
+			(width 0.2)
+			(type default)
+		)
+		(layer "Edge.Cuts")
+	)
+	(gr_arc
+		(start 234.907196 113.5)
+		(mid 234.028516 115.621319)
+		(end 231.907196 116.5)
+		(stroke
+			(width 0.2)
+			(type default)
+		)
+		(layer "Edge.Cuts")
+	)
+	(gr_arc
+		(start 231.907196 58)
+		(mid 234.028519 58.878678)
+		(end 234.907196 61)
+		(stroke
+			(width 0.2)
+			(type default)
+		)
+		(layer "Edge.Cuts")
+	)
+	(gr_line
+		(start 85.907196 113.5)
+		(end 85.907196 61)
+		(stroke
+			(width 0.2)
+			(type default)
+		)
+		(layer "Edge.Cuts")
+	)
+	(gr_arc
+		(start 85.907196 61)
+		(mid 86.785876 58.87868)
+		(end 88.907196 58)
+		(stroke
+			(width 0.2)
+			(type default)
+		)
+		(layer "Edge.Cuts")
+	)
+	(gr_arc
+		(start 88.907196 116.5)
+		(mid 86.785878 115.621319)
+		(end 85.907196 113.5)
 		(stroke
-			(width 0.05)
+			(width 0.2)
 			(type default)
 		)
-		(fill no)
 		(layer "Edge.Cuts")
 	)

Commit message: labels for outputs + new gerbers
Parts:
- added LOGO1: LHRS, UTSVT_Logos:LHRs_LOGO, F.Cu at (219.6, 61.7)
Other:
- board text added: "LV Distribution PCB Surabhi K LHRS 2025"
