File: LV-Distribution/PS-LVDistributionPCB.kicad_sch (KiCad schematic)
At the start: 6 parts, among them J15 Conn_01x20

Commit message: redo traces trial 1
Parts:
- added J16: MX150_02x10_RightAngle, UTSVT_Connectors:CONN_SD-75900-001_2X10_MOL, symbol utsvt_connectors:MX150_02x10_RightAngle
- added J17: MX150_02x10_RightAngle, footprints:CONN_SD-34829-001_20_ST_MOL, symbol utsvt_connectors:MX150_02x10_RightAngle
Connections:
- net GND: now also J16.15, J16.16, J16.17, J16.18, J16.19, J16.20, J17.15, J17.16, J17.17, J17.18, J17.19, J17.20
- net P1: now also J16.1 (+24V), J17.1 (+24V)
- net P10: now also J16.10, J17.10
- net P11: now also J16.11 (GND), J17.11 (GND)
- net P12: now also J16.12 (CANH_OUT), J17.12 (CANH_OUT)
- net P2: now also J16.2 (CANH_IN), J17.2 (CANH_IN)
- net P3: now also J16.3 (CANL_IN), J17.3 (CANL_IN)
- net P4: now also J16.4 (PWR_OUT*), J17.4 (PWR_OUT*)
- net P5: now also J16.5, J17.5
- net P6: now also J16.6, J17.6
- net P7: now also J16.7, J17.7
- net P8: now also J16.8, J17.8
- net P9: now also J16.9, J17.9
- new net P13: J16.13 (CANL_OUT), J17.13 (CANL_OUT)
- new net P14: J16.14 (GND_OUT*), J17.14 (GND_OUT*)
Other:
- removed sheet Power Output
- added sheet Power Output12 (output.kicad_sch)
- added sheet Power Output13 (output.kicad_sch)
- added sheet Power Output14 (output.kicad_sch)

Commit message: better layout but weird 3d stuff
Connections:
- net GND: now also J17.13 (CANL_OUT), J17.14 (GND_OUT*); no longer J17.19, J17.20
- net P1: now also J17.3 (CANL_IN); no longer J17.1 (+24V)
- net P11: now also J17.20; no longer J17.11 (GND)
- net P12: now also J17.19; no longer J17.12 (CANH_OUT)
- net P13: now also J17.7; no longer J17.13 (CANL_OUT)
- net P14: now also J17.6; no longer J17.14 (GND_OUT*)
- net P3: now also J17.1 (+24V); no longer J17.3 (CANL_IN)
- net P4: now also J17.11 (GND); no longer J17.4 (PWR_OUT*)
- net P5: now also J17.12 (CANH_OUT); no longer J17.5
- net P6: now also J17.4 (PWR_OUT*); no longer J17.6
- net P7: now also J17.5; no longer J17.7

Commit message: labels for outputs + new gerbers
Parts:
- removed J15: Conn_01x20, footprints:CONN_SD-34829-001_20_ST_MOL, symbol Connector_Generic:Conn_01x20
- removed J16: MX150_02x10_RightAngle, UTSVT_Connectors:CONN_SD-75900-001_2X10_MOL, symbol utsvt_connectors:MX150_02x10_RightAngle
- added LOGO1: LHRS, UTSVT_Logos:LHRs_LOGO, symbol utsvt_misc:Logo_Placeholder
Other:
- moved on the sheet: H1, H2, H3, H4, H5, J17

Commit message: fixed tvs diode on fuseboard
Parts:
- H1, H2, H3, H4, H5: footprint MountingHole:MountingHole_3.2mm_M3 -> footprints:MountingHole_3.2mm_M3
Changed lines of the file:
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@@
 			)
 		)
-		(property "Footprint" "MountingHole:MountingHole_3.2mm_M3"
+		(property "Footprint" "footprints:MountingHole_3.2mm_M3"
 			(at 207.01 34.29 0)
 			(effects
@@
 			)
 		)
-		(property "Footprint" "MountingHole:MountingHole_3.2mm_M3"
+		(property "Footprint" "footprints:MountingHole_3.2mm_M3"
 			(at 207.01 49.53 0)
 			(effects
@@
 			)
 		)
-		(property "Footprint" "MountingHole:MountingHole_3.2mm_M3"
+		(property "Footprint" "footprints:MountingHole_3.2mm_M3"
 			(at 207.01 55.88 0)
 			(effects
@@
 			)
 		)
-		(property "Footprint" "MountingHole:MountingHole_3.2mm_M3"
+		(property "Footprint" "footprints:MountingHole_3.2mm_M3"
 			(at 207.01 26.67 0)
 			(effects
@@
 			)
 		)
-		(property "Footprint" "MountingHole:MountingHole_3.2mm_M3"
+		(property "Footprint" "footprints:MountingHole_3.2mm_M3"
 			(at 207.01 41.91 0)
 			(effects
