File: LV-Distribution/output.kicad_sch (KiCad schematic)
At the start: 3 parts, among them J1 Conn_01x02

Commit message: lv distribution bom
Parts:
- F1: MANUFACTURER Keystone -> (none); MAXIMUM_PACKAGE_HEIGHT 7.37 mm -> (none); P/N (none) -> 3568; PARTREV C -> (none); SNAPEDA_PN 3568 -> (none); STANDARD Manufacturer Recommendations -> (none)
- J1: P/N (none) -> XT30UPB-M
Changed lines of the file:
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@@
 			)
 		)
-		(property "Datasheet" ""
+		(property "Datasheet" "https://www.mouser.com/datasheet/3/201/1/3568.PDF"
 			(at 52.07 36.83 0)
 			(effects
@@
 			)
 		)
-		(property "Description" ""
+		(property "Description" "SMD fuse holder"
 			(at 52.07 36.83 0)
 			(effects
@@
 			)
 		)
-		(property "PARTREV" "C"
-			(at 52.07 36.83 0)
-			(effects
-				(font
-					(size 1.27 1.27)
-				)
-				(justify bottom)
-				(hide yes)
-			)
-		)
-		(property "MANUFACTURER" "Keystone"
-			(at 52.07 36.83 0)
-			(effects
-				(font
-					(size 1.27 1.27)
-				)
-				(justify bottom)
-				(hide yes)
-			)
-		)
-		(property "SNAPEDA_PN" "3568"
-			(at 52.07 36.83 0)
-			(effects
-				(font
-					(size 1.27 1.27)
-				)
-				(justify bottom)
-				(hide yes)
-			)
-		)
-		(property "MAXIMUM_PACKAGE_HEIGHT" "7.37 mm"
-			(at 52.07 36.83 0)
-			(effects
-				(font
-					(size 1.27 1.27)
-				)
-				(justify bottom)
-				(hide yes)
-			)
-		)
-		(property "STANDARD" "Manufacturer Recommendations"
+		(property "P/N" "3568"
 			(at 52.07 36.83 0)
 			(effects
@@
 			)
 		)
-		(property "Datasheet" "~"
-			(at 69.85 36.83 0)
-			(effects
-				(font
-					(size 1.27 1.27)
-				)
-				(hide yes)
-			)
-		)
-		(property "Description" "Generic connector, single row, 01x02, script generated (kicad-library-utils/schlib/autogen/connector/)"
+		(property "Datasheet" "https://www.tme.com/Document/e5863b891432488e7531b3c4468225ac/XT30PB-M.pdf"
+			(at 69.85 36.83 0)
+			(effects
+				(font
+					(size 1.27 1.27)
+				)
+				(hide yes)
+			)
+		)
+		(property "Description" "XT30 2 pin board mount connector"
+			(at 69.85 36.83 0)
+			(effects
+				(font
+					(size 1.27 1.27)
+				)
+				(hide yes)
+			)
+		)
+		(property "P/N" "XT30UPB-M"
 			(at 69.85 36.83 0)
 			(effects
@@
 			)
 		)
-		(property "Datasheet" "~"
+		(property "Datasheet" "https://www.comchiptech.com/admin/files/product/CPDxx5V0R-HF%20Series%20RevC661473.pdf"
 			(at 38.1 58.42 0)
 			(effects
@@
 			)
 		)
-		(property "Description" "Bidirectional transient-voltage-suppression diode"
+		(property "Description" "0603 TVS diode (rip sorry)"
 			(at 38.1 58.42 0)
 			(effects

Commit message: fixed tvs diode screw you ravi
Parts:
- D1: P/N CPDUC5V0R-HF -> SMBJ30CD-M3/I
Changed lines of the file:
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@@
 			)
 		)
-		(property "Description" "0603 TVS diode (rip sorry)"
+		(property "Description" "SMB TVS diode (rip sorry)"
 			(at 38.1 58.42 0)
 			(effects
@@
 			)
 		)
-		(property "P/N" "CPDUC5V0R-HF "
+		(property "P/N" "SMBJ30CD-M3/I"
 			(at 38.1 58.42 0)
 			(effects

Commit message: fixed tvs diode on fuseboard
Parts:
- D1: footprint Diode_SMD:D_0603_1608Metric -> footprints:D_SMB
Changed lines of the file:
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@@
 			)
 		)
-		(property "Footprint" "Diode_SMD:D_0603_1608Metric"
+		(property "Footprint" "footprints:D_SMB"
 			(at 38.1 58.42 0)
 			(effects
@@
 			)
 		)
-		(property "Description" "SMB TVS diode (rip sorry)"
+		(property "Description" "TVS diode"
 			(at 38.1 58.42 0)
 			(effects
